File: qazlice.kicad_sch (KiCad schematic)
At the start: 0 parts

Commit message: initial schematic
Parts:
- added LED? (x36): YS-SK6812MINI-E, symbol kbd:YS-SK6812MINI-E
- added MX? (x36): MX-NoLED, symbol MX_Alps_Hybrid:MX-NoLED
- added U?: MCP23017_SO, Package_SO:SOIC-28W_7.5x17.9mm_P1.27mm, symbol Interface_Expansion:MCP23017_SO
- added U?: SeeeduinoXIAO, symbol seeeduinoXiao:SeeeduinoXIAO
- added U?: IS31FL3731-QF, Package_DFN_QFN:QFN-28-1EP_4x4mm_P0.4mm_EP2.3x2.3mm, symbol Driver_LED:IS31FL3731-QF
Connections:
- new net: LED?.1 (VDD), LED?.1 (VDD), LED?.1 (VDD), LED?.1 (VDD), LED?.1 (VDD), LED?.1 (VDD), LED?.1 (VDD), LED?.1 (VDD), LED?.1 (VDD), LED?.1 (VDD), LED?.1 (VDD), LED?.1 (VDD), LED?.1 (VDD), LED?.1 (VDD), LED?.1 (VDD), LED?.1 (VDD), LED?.1 (VDD), LED?.1 (VDD), LED?.1 (VDD), LED?.1 (VDD)
- new net: LED?.2 (DOUT), LED?.4 (DIN) (x35)
- new net: LED?.3 (VSS), LED?.3 (VSS), LED?.3 (VSS), LED?.3 (VSS), LED?.3 (VSS), LED?.3 (VSS), LED?.3 (VSS), LED?.3 (VSS), LED?.3 (VSS), LED?.3 (VSS), LED?.3 (VSS), LED?.3 (VSS), LED?.3 (VSS), LED?.3 (VSS), LED?.3 (VSS)
- new net: LED?.1 (VDD), LED?.1 (VDD), LED?.1 (VDD), LED?.1 (VDD), LED?.1 (VDD), LED?.1 (VDD)
- new net: LED?.1 (VDD), LED?.1 (VDD), LED?.1 (VDD), LED?.1 (VDD), LED?.1 (VDD), LED?.1 (VDD), LED?.1 (VDD), LED?.1 (VDD), LED?.1 (VDD), LED?.1 (VDD)
- new net: LED?.3 (VSS), LED?.3 (VSS), LED?.3 (VSS), LED?.3 (VSS), LED?.3 (VSS), LED?.3 (VSS), LED?.3 (VSS), LED?.3 (VSS), LED?.3 (VSS), LED?.3 (VSS), LED?.3 (VSS), LED?.3 (VSS), LED?.3 (VSS), LED?.3 (VSS), LED?.3 (VSS), LED?.3 (VSS), LED?.3 (VSS), LED?.3 (VSS), LED?.3 (VSS), LED?.3 (VSS)
- new net: U?.29 (GND), U?.5 (GND)
- new net COL0: MX?.1 (COL), MX?.1 (COL), MX?.1 (COL), MX?.1 (COL)
- new net COL1: MX?.1 (COL), MX?.1 (COL), MX?.1 (COL)
- new net COL2: MX?.1 (COL), MX?.1 (COL), MX?.1 (COL), MX?.1 (COL)
- new net COL3: MX?.1 (COL), MX?.1 (COL), MX?.1 (COL), MX?.1 (COL)
- new net COL4: MX?.1 (COL), MX?.1 (COL), MX?.1 (COL)
- new net COL5: MX?.1 (COL), MX?.1 (COL), MX?.1 (COL)
- new net COL6: MX?.1 (COL), MX?.1 (COL), MX?.1 (COL), MX?.1 (COL)
- new net COL7: MX?.1 (COL), MX?.1 (COL), MX?.1 (COL), MX?.1 (COL)
- new net COL8: MX?.1 (COL), MX?.1 (COL), MX?.1 (COL)
- new net COL9: MX?.1 (COL), MX?.1 (COL), MX?.1 (COL), MX?.1 (COL)
- new net ROW0: MX?.2 (ROW), MX?.2 (ROW), MX?.2 (ROW), MX?.2 (ROW), MX?.2 (ROW)
- new net ROW1: MX?.2 (ROW), MX?.2 (ROW), MX?.2 (ROW), MX?.2 (ROW), MX?.2 (ROW)
- new net ROW2: MX?.2 (ROW), MX?.2 (ROW), MX?.2 (ROW), MX?.2 (ROW), MX?.2 (ROW)
- new net ROW3: MX?.2 (ROW), MX?.2 (ROW), MX?.2 (ROW)
- new net ROW4: MX?.2 (ROW), MX?.2 (ROW), MX?.2 (ROW), MX?.2 (ROW), MX?.2 (ROW)
- new net ROW5: MX?.2 (ROW), MX?.2 (ROW), MX?.2 (ROW), MX?.2 (ROW), MX?.2 (ROW)
- new net ROW6: MX?.2 (ROW), MX?.2 (ROW), MX?.2 (ROW), MX?.2 (ROW), MX?.2 (ROW)
- new net ROW7: MX?.2 (ROW), MX?.2 (ROW), MX?.2 (ROW)
- no-connect marks 0 -> 1
Other:
- company: (none) -> waffle
- title: (none) -> qazlice
