File: sui.kicad_sch (KiCad schematic)
At the start: 64 parts, among them J1 USB_C_Receptacle, J2 USB_C_Receptacle, U1 SeeeduinoXIAO, U2 SeeeduinoXIAO

Commit message: initial left half
Parts:
- added D23, D24, D25, D26, D27, D28, D29, D30, D31, D32, D33, D34: WS2812B, LED_SMD:LED_WS2812B_PLCC4_5.0x5.0mm_P3.2mm, symbol LED:WS2812B
Connections:
- net +5V: now also D23.1 (VDD), D24.1 (VDD), D25.1 (VDD), D26.1 (VDD), D27.1 (VDD), D28.1 (VDD), D29.1 (VDD), D30.1 (VDD), D31.1 (VDD), D32.1 (VDD), D33.1 (VDD), D34.1 (VDD)
- net COL3_L: now also U1.11 (PA6_A10_D10_MOSI); no longer U1.4 (PA11_A3_D3)
- net GND: now also D23.3 (VSS), D24.3 (VSS), D25.3 (VSS), D26.3 (VSS), D27.3 (VSS), D28.3 (VSS), D29.3 (VSS), D30.3 (VSS), D31.3 (VSS), D32.3 (VSS), D33.3 (VSS), D34.3 (VSS)
- net ROW1_L: now also U1.9 (PA7_A8_D8_SCK); no longer U1.11 (PA6_A10_D10_MOSI)
- net ROW3_L: now also U1.4 (PA11_A3_D3); no longer U1.9 (PA7_A8_D8_SCK)
- net RGB_L: now reaches U1.8 (PB09_A7_D7_RX)
- net RGB_L: now also D27.4 (DIN)
- net RGB_R: now reaches U2.8 (PB09_A7_D7_RX)
- net RGB_R: now also D32.4 (DIN)
- new net: D30.4 (DIN), D31.2 (DOUT)
- new net: D31.4 (DIN), D32.2 (DOUT)
- new net: D23.2 (DOUT), D33.4 (DIN)
- new net: D23.4 (DIN), D24.2 (DOUT)
- new net: D24.4 (DIN), D25.2 (DOUT)
- new net: D28.4 (DIN), D29.2 (DOUT)
- new net: D29.4 (DIN), D30.2 (DOUT)
- new net: D26.4 (DIN), D27.2 (DOUT)
- new net: D28.2 (DOUT), D34.4 (DIN)
- new net: D25.4 (DIN), D26.2 (DOUT)
- no-connect marks 36 -> 38

Commit message: left half complete
Connections:
- net +3V3: no longer names the net of U1.12 (3V3)
- net +3V3: no longer U2.12 (3V3)
- no-connect marks 38 -> 40

Commit message: right half complete
Connections:
- net COL0_R: now also U2.3 (PA10_A2_D2); no longer U2.1 (PA02_A0_D0)
- net COL2_R: now also U2.1 (PA02_A0_D0); no longer U2.3 (PA10_A2_D2)
- net COL3_R: now also U2.11 (PA6_A10_D10_MOSI); no longer U2.4 (PA11_A3_D3)
- net COL4_R: now also U2.9 (PA7_A8_D8_SCK); no longer U2.5 (PA8_A4_D4_SDA)
- net ROW1_R: now also U2.4 (PA11_A3_D3); no longer U2.11 (PA6_A10_D10_MOSI)
- net ROW3_R: now also U2.5 (PA8_A4_D4_SDA); no longer U2.9 (PA7_A8_D8_SCK)
